File: am32_100a_esc.kicad_sch (KiCad schematic)
At the start: 82 parts, among them IC5 DRV8300DPWR, IC6 AS78L05RTR-G1, IC7 L7805ACD2T-TR, IC8 MIC5209-3.3YM-TR, J1 Conn_01x03_Pin, J2 Conn_01x02_Pin, J4 Conn_01x04_Pin, Q13 TPH1R204PB,L1Q, Q14 TPH1R204PB,L1Q, Q15 TPH1R204PB,L1Q, Q16 TPH1R204PB,L1Q, Q17 TPH1R204PB,L1Q, Q18 TPH1R204PB,L1Q, Q19 TPH1R204PB,L1Q, Q20 TPH1R204PB,L1Q, Q21 TPH1R204PB,L1Q, Q22 TPH1R204PB,L1Q, Q23 TPH1R204PB,L1Q, Q24 TPH1R204PB,L1Q, U2 L7809, U4 INA180B2, U6 STM32F051C8Ux

Commit message: ROUTING COMPLETE
Read for production. With Gerber
Parts:
- removed C52, C53: 150uf, Capacitor_THT:CP_Radial_D10.0mm_P5.00mm, symbol Device:C
- added C54, C55, C56, C63, C64, C65: 22uf, Capacitor_SMD:C_1210_3225Metric, symbol Device:C
- added J3, J5, J6, J7: Conn_01x01_Pin, custom_components:capacitor_hole_custom, symbol Connector:Conn_01x01_Pin
- C50, C51: value 150uf -> 1000uf
- H1, H2, H3: footprint MountingHole:MountingHole_3.2mm_M3_Pad -> MountingHole:MountingHole_3.7mm_Pad_Via
- H4, H5: footprint MountingHole:MountingHole_3.2mm_M3_Pad -> MountingHole:MountingHole_4.3mm_M4_Pad_Via
- renumbered LED2 to LED1
Connections:
- net BATT+: now also C54.1, C55.1, C56.1, C63.1, C64.1, C65.1, J3.1 (Pin_1), J6.1 (Pin_1)
- net GND: now also C54.2, C55.2, C56.2, C63.2, C64.2, C65.2, J5.1 (Pin_1), J7.1 (Pin_1)
Other:
- note added: "SMD CAPACITOR BANK"
- note added: "THT CAPACITOR HOLES"
- moved on the sheet: C50, C51

Commit message: Final from my side with drc checked .
Parts:
- BATT+1: renamed from J3; now left out of the parts list
- BATT+2: renamed from J6; now left out of the parts list
- C1, C40: value 0.1uf -> 100nf
- C2, C39, C41: value 0.33uf -> 330nf
- C32, C33: value 100 nf -> 100nf
- C50, C51, J1, J2, J4: now left out of the parts list
- C54, C55, C56, C63, C64, C65: value 22uf -> 4.7uf
- GND1: renamed from J5; now left out of the parts list
- GND2: renamed from J7; now left out of the parts list
- R31, R32, R33, R34, R35, R36, R37, R38, R39, R40, R41, R42: value 5Ω -> 5.1
- renumbered H1 to A1, H2 to B1, H4 to BATT+3, H3 to C3, H5 to GND3

Commit message: re started with routing for better working and removing wrong connections
Parts:
- removed C50, C51: 1000uf, Capacitor_THT:CP_Radial_D10.0mm_P5.00mm, symbol Device:C
Connections:
- net BATT+: now also Q13.5 (D_1), Q13.6 (D_2), Q13.7 (D_3), Q13.8 (D_4), Q13.9 (D_5), Q14.5 (D_1), Q14.6 (D_2), Q14.7 (D_3), Q14.8 (D_4), Q14.9 (D_5), Q15.5 (D_1), Q15.6 (D_2), Q15.7 (D_3), Q15.8 (D_4), Q15.9 (D_5), Q16.5 (D_1), Q16.6 (D_2), Q16.7 (D_3), Q16.8 (D_4), Q16.9 (D_5), Q17.5 (D_1), Q17.6 (D_2), Q17.7 (D_3), Q17.8 (D_4), Q17.9 (D_5), Q18.5 (D_1), Q18.6 (D_2), Q18.7 (D_3), Q18.8 (D_4), Q18.9 (D_5); no longer Q13.1 (S_1), Q13.2 (S_2), Q13.3 (S_3), Q14.1 (S_1), Q14.2 (S_2), Q14.3 (S_3), Q15.1 (S_1), Q15.2 (S_2), Q15.3 (S_3), Q16.1 (S_1), Q16.2 (S_2), Q16.3 (S_3), Q17.1 (S_1), Q17.2 (S_2), Q17.3 (S_3), Q18.1 (S_1), Q18.2 (S_2), Q18.3 (S_3)
- net MOTORA: now also Q13.1 (S_1), Q13.2 (S_2), Q13.3 (S_3), Q16.1 (S_1), Q16.2 (S_2), Q16.3 (S_3); no longer Q13.5 (D_1), Q13.6 (D_2), Q13.7 (D_3), Q13.8 (D_4), Q13.9 (D_5), Q16.5 (D_1), Q16.6 (D_2), Q16.7 (D_3), Q16.8 (D_4), Q16.9 (D_5)
- net MOTORB: now also Q14.1 (S_1), Q14.2 (S_2), Q14.3 (S_3), Q17.1 (S_1), Q17.2 (S_2), Q17.3 (S_3); no longer Q14.5 (D_1), Q14.6 (D_2), Q14.7 (D_3), Q14.8 (D_4), Q14.9 (D_5), Q17.5 (D_1), Q17.6 (D_2), Q17.7 (D_3), Q17.8 (D_4), Q17.9 (D_5)
- net MOTORC: now also Q15.1 (S_1), Q15.2 (S_2), Q15.3 (S_3), Q18.1 (S_1), Q18.2 (S_2), Q18.3 (S_3); no longer Q15.5 (D_1), Q15.6 (D_2), Q15.7 (D_3), Q15.8 (D_4), Q15.9 (D_5), Q18.5 (D_1), Q18.6 (D_2), Q18.7 (D_3), Q18.8 (D_4), Q18.9 (D_5)
Other:
- note removed: "CAPACITOR BANK"
- moved on the sheet: Q13, Q14, Q15, Q16, Q17, Q18, Q19, Q20, Q21, Q22, Q23, Q24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
